File: Hardware/Kicad FIles/mPLC.kicad_pcb (KiCad board)
At the start: 4 copper layers, 100 x 100 mm, 161 parts, among them J1 Connector, USB-TYPE-C-16P, J2 2601-3111, J3 2601-3111, J4 2601-3104, J5 2601-3104, J6 2601-3104, J7 Header, 2.54mm, 1x8P, Male, V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, Q1 HL3400A, Q10 HL3400A, Q11 HL3400A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

Commit message: Add files via upload
Parts:
- added D12: SS56, JLCPCB-Kicad-Footprints:D_SMC, F.Cu at (107.7, 52.8)
- added F1: 1.5A, JLCPCB-Kicad-Footprints:F_1206, F.Cu at (118.4, 54.2)
- moved D3 20.7 mm to (124.0, 65.8), turned to -90 degrees
- moved C8 12.8 mm to (121.7, 78.5), turned to 180 degrees
- moved C9 11.6 mm to (121.7, 81.0), turned to 180 degrees
- moved C10 11.3 mm to (121.7, 83.6), turned to 180 degrees
- moved C17 9.11 mm to (112.3, 73.4), turned to 180 degrees
- moved C3 8.04 mm to (129.5, 59.2), turned to 180 degrees
- moved C13 7.43 mm to (112.3, 83.6), turned to 180 degrees
- moved U2 7.13 mm to (127.8, 55.0), turned to 180 degrees
- moved C16 6.09 mm to (112.3, 75.9), turned to 180 degrees
- moved C5 6.08 mm to (121.9, 54.6), turned to 90 degrees
- moved R3 5.48 mm to (131.1, 62.7)
- moved C1 5.46 mm to (104.2, 69.6), turned to 90 degrees
- moved R4 5.41 mm to (128.7, 62.7)
- moved C14 4.89 mm to (112.3, 81.0), turned to 180 degrees
- moved C6 4.76 mm to (121.7, 73.4), turned to 180 degrees
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Connections:
- C4 pad 1: Net-(J6-1_1) -> Net-(U2-VIN)
- C5 pad 1: Net-(J6-1_1) -> Net-(U2-VIN)
- U2 pad 7: Net-(J6-1_1) -> Net-(U2-VIN)
Routing:
- net GND: track 268.3 -> 205.0 mm, vias 128 -> 141
- net Net-(U2-VIN): track 0.00 -> 25.3 mm
- net Net-(J6-1_1): track 38.1 -> 21.0 mm
- net +5V: track 47.7 -> 37.5 mm
- net +10V: track 96.4 -> 105.1 mm, vias 0 -> 2
- net Net-(U2-VSENSE): track 4.25 -> 12.8 mm
- net Net-(U2-PH): track 21.9 -> 16.0 mm
- net +3V3: track 75.5 -> 74.3 mm
