File: Hardware/Kicad FIles/mPLC.kicad_sch (KiCad schematic)
At the start: 0 parts

Commit message: Add files via upload
Changed lines of the file:
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@@
 	(paper "A4")
 	(sheet
-		(at 41.91 118.11)
-		(size 38.1 31.75)
+		(at 153.67 39.37)
+		(size 30.48 20.32)
 		(fields_autoplaced yes)
 		(stroke
@@
 		)
 		(property "Sheetname" "Analog"
-			(at 41.91 117.3984 0)
+			(at 153.67 38.6584 0)
 			(effects
 				(font
@@
 		)
 		(property "Sheetfile" "Analog.kicad_sch"
-			(at 41.91 150.4446 0)
+			(at 153.67 60.2746 0)
 			(effects
 				(font
@@
 		)
 		(instances
-			(project "CNC"
+			(project "mPLC"
 				(path "/9ed7c920-cc63-4d6b-a8e8-76de1b6d60db"
 					(page "6")
@@
 	)
 	(sheet
-		(at 172.72 48.26)
-		(size 46.99 27.94)
+		(at 113.03 39.37)
+		(size 33.02 20.32)
 		(fields_autoplaced yes)
 		(stroke
@@
 		)
 		(property "Sheetname" "IO"
-			(at 172.72 47.5484 0)
+			(at 113.03 38.6584 0)
 			(effects
 				(font
@@
 		)
 		(property "Sheetfile" "IO.kicad_sch"
-			(at 172.72 76.7846 0)
+			(at 113.03 60.2746 0)
 			(effects
 				(font
@@
 		)
 		(instances
-			(project "CNC"
+			(project "mPLC"
 				(path "/9ed7c920-cc63-4d6b-a8e8-76de1b6d60db"
 					(page "4")
@@
 	(sheet
 		(at 29.21 39.37)
-		(size 46.99 36.83)
+		(size 33.02 20.32)
 		(fields_autoplaced yes)
 		(stroke
@@
 		)
 		(property "Sheetfile" "PUSB.kicad_sch"
-			(at 29.21 76.7846 0)
+			(at 29.21 60.2746 0)
 			(effects
 				(font
@@
 		)
 		(instances
-			(project "CNC"
+			(project "mPLC"
 				(path "/9ed7c920-cc63-4d6b-a8e8-76de1b6d60db"
 					(page "2")
@@
 	)
 	(sheet
-		(at 95.25 44.45)
-		(size 46.99 27.94)
+		(at 69.85 39.37)
+		(size 34.29 20.32)
 		(fields_autoplaced yes)
 		(stroke
@@
 		)
 		(property "Sheetname" "MCU"
-			(at 95.25 43.7384 0)
+			(at 69.85 38.6584 0)
 			(effects
 				(font
@@
 		)
 		(property "Sheetfile" "MCU.kicad_sch"
-			(at 95.25 72.9746 0)
+			(at 69.85 60.2746 0)
 			(effects
 				(font
@@
 		)
 		(instances
-			(project "CNC"
+			(project "mPLC"
 				(path "/9ed7c920-cc63-4d6b-a8e8-76de1b6d60db"
 					(page "3")
